Commit message: Task A3 completed. Parameter file created and collision is as per the parameter file. Color argument also added.

File: nuturtle_description/urdf/turtlebot3_burger.urdf.xacro (robot description, xacro)
@@ -2,5 +2,11 @@
 <robot name="turtlebot3_burger"
   xmlns:xacro="http://ros.org/wiki/xacro">
+  <xacro:property name="diff_params" value="$(find nuturtle_description)/config/diff_prams.yaml" />
+  <xacro:property name="props" value="${xacro.load_yaml(diff_params)['/**']['ros__parameters']}" />
+  <xacro:property name="wheel_radius" value="${props['wheel_radius']}" />
+  <xacro:property name="track_width" value="${props['track_width']}" />
+  <xacro:property name="collision_radius" value="${props['collision_radius']}" />
   <!-- <xacro:include filename="$(find turtlebot3_description)/urdf/common_properties.urdf"/> -->
+  <xacro:property name="color" value="$(arg color)"/>
   <!-- Init colour -->
   <material name="black">
@@ -34,4 +40,7 @@
     <color rgba="1.0 1.0 1.0 1.0"/>
   </material>
+  <material name="purple">
+    <color rgba="0.3 0.16 0.52 1.0"/>
+  </material>
   <link name="base_footprint"/>
   <joint name="base_joint" type="fixed">
@@ -46,10 +55,15 @@
         <mesh filename="file://$(find nuturtle_description)/meshes/burger_base.stl" scale="0.001 0.001 0.001"/>
       </geometry>
-      <material name="light_black"/>
+      <material name="${color}"/>
     </visual>
     <collision>
       <origin xyz="-0.032 0 0.070" rpy="0 0 0"/>
       <geometry>
+        <xacro:if value="${collision_radius &gt; 0}">
+          <cylinder length="0.140" radius="${track_width/2}"/>
+        </xacro:if>
+       <xacro:if value="${collision_radius &lt;= 0}">
         <box size="0.140 0.140 0.143"/>
+       </xacro:if>
       </geometry>
     </collision>
@@ -63,5 +77,5 @@
     <parent link="base_link"/>
     <child link="wheel_left_link"/>
-    <origin xyz="0.0 0.08 0.023" rpy="-1.57 0 0"/>
+    <origin xyz="0.0 ${track_width/2} 0.023" rpy="-1.57 0 0"/>
     <axis xyz="0 0 1"/>
   </joint>
@@ -77,5 +91,5 @@
       <origin xyz="0 0 0" rpy="0 0 0"/>
       <geometry>
-        <cylinder length="0.018" radius="0.033"/>
+        <cylinder length="0.018" radius="${wheel_radius}"/>
       </geometry>
     </collision>
@@ -89,5 +103,5 @@
     <parent link="base_link"/>
     <child link="wheel_right_link"/>
-    <origin xyz="0.0 -0.080 0.023" rpy="-1.57 0 0"/>
+    <origin xyz="0.0 ${track_width/-2} 0.023" rpy="-1.57 0 0"/>
     <axis xyz="0 0 1"/>
   </joint>
@@ -103,5 +117,5 @@
       <origin xyz="0 0 0" rpy="0 0 0"/>
       <geometry>
-        <cylinder length="0.018" radius="0.033"/>
+        <cylinder length="0.018" radius="${wheel_radius}"/>
       </geometry>
     </collision>
